File: ER-TFT035-6_LCD_Interface.kicad_sch (KiCad schematic)
At the start: 9 parts, among them Q101 IRLML0040TR, X101 62684-502100ALF

Commit message: Move encoder into its own sheet. Replace with MPG/Encoder combo.
Parts:
- JP301: renamed from JP101; footprint (none) -> Jumper:SolderJumper-3_P2.0mm_Open_TrianglePad1.0x1.5mm_NumberLabels
- JP302: renamed from JP102; footprint (none) -> Jumper:SolderJumper-3_P2.0mm_Open_TrianglePad1.0x1.5mm_NumberLabels
- Q301: renamed from Q101; footprint (none) -> Package_TO_SOT_SMD:SOT-23
- R301: renamed from R104; footprint (none) -> Resistor_SMD:R_0805_2012Metric_Pad1.20x1.40mm_HandSolder
- R302: renamed from R102; footprint (none) -> Resistor_SMD:R_0805_2012Metric_Pad1.20x1.40mm_HandSolder
- R303: renamed from R101; footprint (none) -> Resistor_SMD:R_0805_2012Metric_Pad1.20x1.40mm_HandSolder
- R304: renamed from R103; footprint (none) -> Resistor_SMD:R_0805_2012Metric_Pad1.20x1.40mm_HandSolder
- X301: renamed from X101; footprint CONN50_62684-502100ALF_FCI -> MarcoK:62684-502100ALF
- renumbered DP101 to DP301
Changed lines of the file:
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@@
     (effects (font (size 0.9906 0.9906)) (justify left))
   )
-  (symbol (lib_id "Connector:Conn_01x15_Female") (at 185.42 92.71 180)
-    (in_bom yes) (on_board yes)
-    (property "Reference" "DP101" (id 0) (at 184.7088 93.3704 0)
+  (symbol (lib_id "Connector:Conn_01x15_Female") (at 185.42 92.71 180) (unit 1)
+    (in_bom yes) (on_board yes)
+    (property "Reference" "DP301" (id 0) (at 184.7088 93.3704 0)
       (effects (font (size 1.27 1.27)) (justify left))
     )
@@
   (symbol (lib_id "power:GND") (at 204.47 115.57 0) (unit 1)
     (in_bom yes) (on_board yes)
-    (property "Reference" "#PWR?" (id 0) (at 204.47 121.92 0)
+    (property "Reference" "#PWR0312" (id 0) (at 204.47 121.92 0)
       (effects (font (size 1.27 1.27)) hide)
     )
@@
   (symbol (lib_id "Device:R") (at 63.5 35.56 270) (unit 1)
     (in_bom yes) (on_board yes)
-    (property "Reference" "R104" (id 0) (at 63.5 30.3022 90))
+    (property "Reference" "R301" (id 0) (at 63.5 30.3022 90))
     (property "Value" "10" (id 1) (at 63.5 32.6136 90))
-    (property "Footprint" "" (id 2) (at 63.5 33.782 90)
+    (property "Footprint" "Resistor_SMD:R_0805_2012Metric_Pad1.20x1.40mm_HandSolder" (id 2) (at 63.5 33.782 90)
       (effects (font (size 1.27 1.27)) hide)
     )
@@
   (symbol (lib_id "power:+3V3") (at 73.66 25.4 0) (unit 1)
     (in_bom yes) (on_board yes)
-    (property "Reference" "#PWR?" (id 0) (at 73.66 29.21 0)
+    (property "Reference" "#PWR0307" (id 0) (at 73.66 29.21 0)
       (effects (font (size 1.27 1.27)) hide)
     )
@@
     (pin "1")
   )
-  (symbol (lib_id "MarcoK:IRLML0040TR") (at 127 41.91 0)
-    (in_bom yes) (on_board yes)
-    (property "Reference" "Q101" (id 0) (at 131.1402 41.91 0)
+  (symbol (lib_id "MarcoK:IRLML0040TR") (at 127 41.91 0) (unit 1)
+    (in_bom yes) (on_board yes)
+    (property "Reference" "Q301" (id 0) (at 131.1402 41.91 0)
       (effects (font (size 1.4986 1.4986)) (justify left))
     )
@@
       (effects (font (size 1.4986 1.4986)) (justify left) hide)
     )
-    (property "Footprint" "" (id 2) (at 127 41.91 0)
+    (property "Footprint" "Package_TO_SOT_SMD:SOT-23" (id 2) (at 127 41.91 0)
       (effects (font (size 0.254 0.254)) hide)
     )
@@
     (pin "3")
   )
-  (symbol (lib_id "power:GND") (at 127 52.07 0)
-    (in_bom yes) (on_board yes)
-    (property "Reference" "#PWR?" (id 0) (at 127 58.42 0)
+  (symbol (lib_id "power:GND") (at 127 52.07 0) (unit 1)
+    (in_bom yes) (on_board yes)
+    (property "Reference" "#PWR0311" (id 0) (at 127 58.42 0)
       (effects (font (size 1.27 1.27)) hide)
     )
@@
   (symbol (lib_id "Device:R") (at 91.44 133.35 270) (unit 1)
     (in_bom yes) (on_board yes)
-    (property "Reference" "R101" (id 0) (at 91.44 128.0922 90))
+    (property "Reference" "R303" (id 0) (at 91.44 128.0922 90))
     (property "Value" "10" (id 1) (at 91.44 130.4036 90))
-    (property "Footprint" "" (id 2) (at 91.44 131.572 90)
+    (property "Footprint" "Resistor_SMD:R_0805_2012Metric_Pad1.20x1.40mm_HandSolder" (id 2) (at 91.44 131.572 90)
       (effects (font (size 1.27 1.27)) hide)
     )
@@
   (symbol (lib_id "Device:R") (at 71.12 128.27 270) (unit 1)
     (in_bom yes) (on_board yes)
-    (property "Reference" "R102" (id 0) (at 71.12 123.0122 90))
+    (property "Reference" "R302" (id 0) (at 71.12 123.0122 90))
     (property "Value" "10" (id 1) (at 71.12 125.3236 90))
-    (property "Footprint" "" (id 2) (at 71.12 126.492 90)
+    (property "Footprint" "Resistor_SMD:R_0805_2012Metric_Pad1.20x1.40mm_HandSolder" (id 2) (at 71.12 126.492 90)
       (effects (font (size 1.27 1.27)) hide)
     )
@@
   (symbol (lib_id "Device:R") (at 113.03 134.62 0) (mirror x) (unit 1)
     (in_bom yes) (on_board yes)
-    (property "Reference" "R103" (id 0) (at 107.7722 134.62 90))
+    (property "Reference" "R304" (id 0) (at 107.7722 134.62 90))
     (property "Value" "10K" (id 1) (at 110.0836 134.62 90))
-    (property "Footprint" "" (id 2) (at 111.252 134.62 90)
+    (property "Footprint" "Resistor_SMD:R_0805_2012Metric_Pad1.20x1.40mm_HandSolder" (id 2) (at 111.252 134.62 90)
       (effects (font (size 1.27 1.27)) hide)
     )
@@
   (symbol (lib_id "Jumper:SolderJumper_3_Bridged12") (at 73.66 35.56 270) (unit 1)
     (in_bom yes) (on_board yes)
-    (property "Reference" "JP101" (id 0) (at 75.3872 35.56 90)
+    (property "Reference" "JP301" (id 0) (at 75.3872 35.56 90)
       (effects (font (size 1.27 1.27)) (justify left))
     )
@@
       (effects (font (size 1.27 1.27)) hide)
     )
-    (property "Footprint" "" (id 2) (at 73.66 35.56 0)
+    (property "Footprint" "Jumper:SolderJumper-3_P2.0mm_Open_TrianglePad1.0x1.5mm_NumberLabels" (id 2) (at 73.66 35.56 0)
       (effects (font (size 1.27 1.27)) hide)
     )
@@
   (symbol (lib_id "Jumper:SolderJumper_3_Bridged12") (at 97.79 35.56 270) (unit 1)
     (in_bom yes) (on_board yes)
-    (property "Reference" "JP102" (id 0) (at 99.5172 35.56 90)
+    (property "Reference" "JP302" (id 0) (at 99.5172 35.56 90)
       (effects (font (size 1.27 1.27)) (justify left))
     )
@@
       (effects (font (size 1.27 1.27)) (justify left) hide)
     )
-    (property "Footprint" "" (id 2) (at 97.79 35.56 0)
+    (property "Footprint" "Jumper:SolderJumper-3_P2.0mm_Open_TrianglePad1.0x1.5mm_NumberLabels" (id 2) (at 97.79 35.56 0)
       (effects (font (size 1.27 1.27)) hide)
     )
@@
   (symbol (lib_id "power:+3V3") (at 210.82 88.9 0) (unit 1)
     (in_bom yes) (on_board yes)
-    (property "Reference" "#PWR?" (id 0) (at 210.82 92.71 0)
+    (property "Reference" "#PWR0313" (id 0) (at 210.82 92.71 0)
       (effects (font (size 1.27 1.27)) hide)
     )
@@
   (symbol (lib_id "MarcoK:62684-502100ALF") (at 53.34 44.45 0) (mirror y) (unit 1)
     (in_bom yes) (on_board yes)
-    (property "Reference" "X101" (id 0) (at 39.9288 105.3338 0)
+    (property "Reference" "X301" (id 0) (at 39.9288 105.3338 0)
       (effects (font (size 1.524 1.524)) (justify left))
     )
@@
       (effects (font (size 1.524 1.524)) (justify left))
     )
-    (property "Footprint" "CONN50_62684-502100ALF_FCI" (id 2) (at 43.18 106.934 0)
+    (property "Footprint" "MarcoK:62684-502100ALF" (id 2) (at 43.18 106.934 0)
       (effects (font (size 1.524 1.524)) hide)
     )
@@
   (symbol (lib_id "power:+3V3") (at 68.58 59.69 0) (unit 1)
     (in_bom yes) (on_board yes)
-    (property "Reference" "#PWR?" (id 0) (at 68.58 63.5 0)
+    (property "Reference" "#PWR0303" (id 0) (at 68.58 63.5 0)
       (effects (font (size 1.27 1.27)) hide)
     )
@@
     (pin "1")
   )
-  (symbol (lib_id "power:GND") (at 68.58 72.39 0)
-    (in_bom yes) (on_board yes)
-    (property "Reference" "#PWR?" (id 0) (at 68.58 78.74 0)
+  (symbol (lib_id "power:GND") (at 68.58 72.39 0) (unit 1)
+    (in_bom yes) (on_board yes)
+    (property "Reference" "#PWR0304" (id 0) (at 68.58 78.74 0)
       (effects (font (size 1.27 1.27)) hide)
     )
@@
   (symbol (lib_id "power:+3V3") (at 78.74 73.66 0) (unit 1)
     (in_bom yes) (on_board yes)
-    (property "Reference" "#PWR?" (id 0) (at 78.74 77.47 0)
+    (property "Reference" "#PWR0308" (id 0) (at 78.74 77.47 0)
       (effects (font (size 1.27 1.27)) hide)
     )
@@
   (symbol (lib_id "power:+3V3") (at 86.36 120.65 0) (unit 1)
     (in_bom yes) (on_board yes)
-    (property "Reference" "#PWR?" (id 0) (at 86.36 124.46 0)
+    (property "Reference" "#PWR0309" (id 0) (at 86.36 124.46 0)
       (effects (font (size 1.27 1.27)) hide)
     )
@@
   (symbol (lib_id "power:+3V3") (at 113.03 120.65 0) (unit 1)
     (in_bom yes) (on_board yes)
-    (property "Reference" "#PWR?" (id 0) (at 113.03 124.46 0)
+    (property "Reference" "#PWR0310" (id 0) (at 113.03 124.46 0)
       (effects (font (size 1.27 1.27)) hide)
     )
@@
   (symbol (lib_id "power:+3V3") (at 62.23 144.78 0) (unit 1)
     (in_bom yes) (on_board yes)
-    (property "Reference" "#PWR?" (id 0) (at 62.23 148.59 0)
+    (property "Reference" "#PWR0302" (id 0) (at 62.23 148.59 0)
       (effects (font (size 1.27 1.27)) hide)
     )
@@
     (pin "1")
   )
-  (symbol (lib_id "power:GND") (at 68.58 152.4 0)
-    (in_bom yes) (on_board yes)
-    (property "Reference" "#PWR?" (id 0) (at 68.58 158.75 0)
+  (symbol (lib_id "power:GND") (at 68.58 152.4 0) (unit 1)
+    (in_bom yes) (on_board yes)
+    (property "Reference" "#PWR0306" (id 0) (at 68.58 158.75 0)
       (effects (font (size 1.27 1.27)) hide)
     )
@@
     (pin "1")
   )
-  (symbol (lib_id "power:GND") (at 57.15 172.72 0)
-    (in_bom yes) (on_board yes)
-    (property "Reference" "#PWR?" (id 0) (at 57.15 179.07 0)
+  (symbol (lib_id "power:GND") (at 57.15 172.72 0) (unit 1)
+    (in_bom yes) (on_board yes)
+    (property "Reference" "#PWR0301" (id 0) (at 57.15 179.07 0)
       (effects (font (size 1.27 1.27)) hide)
     )
@@
     (pin "1")
   )
-  (symbol (lib_id "power:GND") (at 68.58 102.87 0)
-    (in_bom yes) (on_board yes)
-    (property "Reference" "#PWR?" (id 0) (at 68.58 109.22 0)
-      (effects (font (size 1.27 1.27)) hide)
-    )
+  (symbol (lib_id "power:GND") (at 68.58 102.87 0) (unit 1)
+    (in_bom yes) (on_board yes)
+    (property "Reference" "#PWR0305" (id 0) (at 68.58 109.22 0)
+      (effects (font (size 1.27 1.27)) hide)
+    )

Commit message: Added the MPG. Switched tactile button model. Added JLC design rules.
Parts:
- DP301: footprint MarcoK:BUY_LCD_TFT035-6_320x480-BO -> Connector_PinSocket_2.54mm:PinSocket_1x15_P2.54mm_Vertical
- X301: footprint MarcoK:62684-502100ALF -> MarcoK:TFT_3.5IN_320X480_50PIN_BUY_DISPLAY_ER-TFT035-6
Changed lines of the file:
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@@
       (effects (font (size 1.27 1.27)) (justify left) hide)
     )
-    (property "Footprint" "MarcoK:BUY_LCD_TFT035-6_320x480-BO" (id 2) (at 185.42 92.71 0)
+    (property "Footprint" "Connector_PinSocket_2.54mm:PinSocket_1x15_P2.54mm_Vertical" (id 2) (at 185.42 92.71 0)
       (effects (font (size 1.27 1.27)) hide)
     )
@@
       (effects (font (size 1.524 1.524)) (justify left))
     )
-    (property "Footprint" "MarcoK:62684-502100ALF" (id 2) (at 43.18 106.934 0)
+    (property "Footprint" "MarcoK:TFT_3.5IN_320X480_50PIN_BUY_DISPLAY_ER-TFT035-6" (id 2) (at 43.18 106.934 0)
       (effects (font (size 1.524 1.524)) hide)
     )
