File: XCarveDRO.kicad_pcb (KiCad board)
At the start: 2 copper layers, 200 x 150 mm, 100 parts, among them J101 USB_B, J102 Jack-DC, J103 USB_A, Q101 FDN340P, Q102 FDN340P, Q301 IRLML0040TR, SW101 SW_DPST_x2, SW103 SEL1, SW104 SEL2, SW201 SWITCH_FSM4JSMATR_TYC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

Commit message: Update 3D components.
Parts:
- REF** (x11): value MountingHole_3.2mm_M3 -> MountingHole_3.2mm_M3_Pad; footprint MountingHole:MountingHole_3.2mm_M3 -> MountingHole:MountingHole_3.2mm_M3_Pad
Other:
- rule pad_to_mask_clearance: 0.05 -> 0
